Commit message: pushing the intermediate version of the project

File: notebooks/room.urdf (robot description, URDF)
Before this commit: robot lab_room, 5 links, 4 joints
Links:
- link wall_e: geometry collision box size=0.1 10 3; visual box size=0.1 10 3
- link wall_n: geometry collision box size=10 0.1 3; visual box size=10 0.1 3
- link wall_s: geometry collision box size=10 0.1 3; visual box size=10 0.1 3
- link wall_w: geometry collision box size=0.1 10 3; visual box size=0.1 10 3
